File: Hardware/PWM_Regulator.kicad_pcb (KiCad board)
At the start: 2 copper layers, 55 x 16 mm, 51 parts

Commit message: Трассировка завершена.
Parts:
- moved C15 6.29 mm to (148.2, 60.0), turned to 90 degrees
- moved C10 3.25 mm to (126.5, 55.2), turned to 270 degrees
- moved C11 2.75 mm to (126.5, 52.2), turned to 90 degrees
- moved C6 1.75 mm to (139.5, 54.5)
- moved C8 1.75 mm to (137.8, 54.5)
- moved fus1 1.52 mm to (130.5, 51.0)
- moved C14 1.12 mm to (147.5, 63.0)
- moved VD5 1.03 mm to (148.2, 56.0)
- moved VD6 1.00 mm to (147.5, 65.0)
- moved DA1 0.50 mm to (116.0, 54.0)
- moved C13 0.25 mm to (124.8, 52.2)
- moved R8 0.25 mm to (124.8, 55.2)
- moved XS1 0.25 mm to (144.5, 51.5)
- turned SB1 to 180 degrees
- turned SB2 to 180 degrees
Routing:
- net GND: track 0.00 -> 148.3 mm, vias 0 -> 15
- net +3.3V: track 0.00 -> 78.8 mm, vias 0 -> 3
- net +12Vin: track 0.00 -> 78.0 mm
- net GNDP: track 0.00 -> 67.5 mm, vias 0 -> 7
- net /+MSU_PWR: track 0.00 -> 38.5 mm
- net /ADC: track 0.00 -> 31.3 mm, vias 0 -> 2
- net /PWM_OUT: track 0.00 -> 19.0 mm
- net /PWM: track 0.00 -> 17.6 mm, vias 0 -> 2
- net /USER: track 0.00 -> 16.6 mm, vias 0 -> 3
- net /SWCLK: track 0.00 -> 16.3 mm, vias 0 -> 1
- net /EN_WKUP: track 0.00 -> 15.4 mm
- net /BTN2: track 0.00 -> 14.9 mm, vias 0 -> 1
- net /UART_TX: track 0.00 -> 13.0 mm, vias 0 -> 1
- net +12V: track 0.00 -> 12.9 mm, vias 0 -> 1
- net /UART_RX: track 0.00 -> 11.0 mm, vias 0 -> 1
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- added copper zone on B.Cu, net GND
- added copper zone on F.Cu, net GND

Commit message: Доделано заземление, расставлены надписи
Parts:
- DA2: value LP2985-xx -> LP2985-33
- moved C1 0.79 mm to (105.0, 55.0)
- moved HL1 0.50 mm to (104.5, 63.0)
- moved R5 0.50 mm to (108.5, 63.0)
Routing:
- net GND: track 148.3 -> 230.7 mm, vias 15 -> 34
- net GNDP: track 67.5 -> 62.7 mm, vias 7 -> 3
- net +12Vin: track 78.0 -> 80.3 mm
- net +3.3V: track 78.8 -> 81.1 mm
- net Net-(R2-Pad2): track 7.04 -> 8.66 mm
- net /+MSU_PWR: track 38.5 -> 39.8 mm
- net /PWM_OUT: track 19.0 -> 20.2 mm
- net /GNDin: track 9.21 -> 8.09 mm

Commit message: работа завершена
Other:
- board text added: "12Vin"
- board text added: "ADCin"
- board text added: "OUT"
- board text added: "instead 2985"
- board text added: "~EN"
- board text added: "«PWM Regulator»"
Changed lines of the file:
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@@
 (kicad_pcb (version 20171130) (host pcbnew "(5.1.7)-1")
   (general
-    (thickness 1.6)
-    (drawings 56)
+    (thickness 1)
+    (drawings 63)
     (tracks 934)
     (zones 0)
@@
     (aux_axis_origin 155 66)
     (grid_origin 100 50)
-    (visible_elements 7FFFFF3F)
+    (visible_elements 7FFFFF7F)
     (pcbplotparams
       (layerselection 0x010f0_ffffffff)
@@
     (at 116 54 90)
     (attr smd)
-    (fp_text reference DA1 (at 0 0.5 90) (layer B.SilkS)
+    (fp_text reference DA1 (at 0 -1.25 90) (layer B.SilkS)
       (effects (font (size 0.6 0.6) (thickness 0.15)) (justify mirror))
     )
-    (fp_text value TLV1117-33 (at 0 -0.75 90) (layer B.SilkS)
+    (fp_text value TLV1117-33 (at 0 -0.25 90) (layer B.SilkS)
       (effects (font (size 0.6 0.6) (thickness 0.15)) (justify mirror))
     )
@@
       (effects (font (size 0.8 0.6) (thickness 0.15)) (justify mirror))
     )
-    (fp_text value Up (at 0 3.175 180) (layer B.SilkS)
+    (fp_text value Up (at -4 0 270) (layer B.SilkS)
       (effects (font (size 1 0.8) (thickness 0.15)) (justify mirror))
     )
@@
       (effects (font (size 0.8 0.6) (thickness 0.15)) (justify mirror))
     )
-    (fp_text value Down (at 0 3.175 180) (layer B.SilkS)
+    (fp_text value Down (at -4.5 0 270) (layer B.SilkS)
       (effects (font (size 1 0.8) (thickness 0.15)) (justify mirror))
     )
@@
       (effects (font (size 1.5 1.5) (thickness 0.3)))
     )
-    (fp_text user + (at -1.25 -1.75 270) (layer B.SilkS)
+    (fp_text user + (at -3.5 0 270) (layer B.SilkS)
       (effects (font (size 1.5 1.5) (thickness 0.3)) (justify mirror))
     )
-    (fp_text user - (at 1.25 -1.75 270) (layer B.SilkS)
+    (fp_text user - (at 3.5 0 270) (layer B.SilkS)
       (effects (font (size 1.5 1.5) (thickness 0.3)) (justify mirror))
     )
@@
       (effects (font (size 0.8 0.8) (thickness 0.15)))
     )
-    (fp_text user VCC (at -3.302 -2.159) (layer B.SilkS)
+    (fp_text user VCC (at -2.488 -2.982 90) (layer B.SilkS)
       (effects (font (size 1 1) (thickness 0.15)) (justify mirror))
     )
-    (fp_text user GND (at 0 -2.159) (layer B.SilkS)
+    (fp_text user GND (at 0.012 -2.982 90) (layer B.SilkS)
       (effects (font (size 1 1) (thickness 0.15)) (justify mirror))
     )
-    (fp_text user OUT (at 3.302 -2.159) (layer B.SilkS)
+    (fp_text user OUT (at 2.512 -2.982 90) (layer B.SilkS)
       (effects (font (size 1 1) (thickness 0.15)) (justify mirror))
     )
@@
       (net 19 /UART_RX))
   )
+  (gr_text "instead 2985" (at 117 54 90) (layer B.SilkS)
+    (effects (font (size 0.6 0.6) (thickness 0.15)) (justify mirror))
+  )
+  (gr_text "«PWM Regulator»" (at 145.75 64) (layer B.SilkS)
+    (effects (font (size 1.2 1.2) (thickness 0.2) italic) (justify mirror))
+  )
+  (gr_text OUT (at 148 58 90) (layer B.SilkS)
+    (effects (font (size 1.2 1.2) (thickness 0.2)) (justify mirror))
+  )
+  (gr_text 12Vin (at 103.75 58 270) (layer B.SilkS)
+    (effects (font (size 1.2 1.2) (thickness 0.2)) (justify mirror))
+  )
+  (gr_text ~EN (at 123.5 62.25 90) (layer B.SilkS)
+    (effects (font (size 1 0.8) (thickness 0.15)) (justify mirror))
+  )
+  (gr_text GND (at 126 62 90) (layer B.SilkS)
+    (effects (font (size 1 0.8) (thickness 0.15)) (justify mirror))
+  )
+  (gr_text ADCin (at 119.5 62.5) (layer B.SilkS)
+    (effects (font (size 1 0.8) (thickness 0.15)) (justify mirror))
+  )
   (gr_line (start 141.6 57.2) (end 141.7 52.8) (angle 90) (layer F.SilkS) (width 0.15))
   (gr_line (start 139.7 58.7) (end 141.6 57.2) (angle 90) (layer F.SilkS) (width 0.15))
@@
     (effects (font (size 1 0.8) (thickness 0.15)) (justify mirror))
   )
-  (gr_text GND (at 151 55.75) (layer B.SilkS)
+  (gr_text GND (at 151 55.5) (layer B.SilkS)
     (effects (font (size 1 0.8) (thickness 0.15)) (justify mirror))
   )
@@
     (effects (font (size 1 0.8) (thickness 0.15)))
   )
-  (gr_text GND (at 151 55.75) (layer F.SilkS)
+  (gr_text GND (at 151 55.5) (layer F.SilkS)
     (effects (font (size 1 0.8) (thickness 0.15)))
   )
