File: Hardware/GameTimer.sch (KiCad schematic (older format))
At the start: 68 parts

Commit message: Игровой таймер: расстановка компонентов наяата
Parts:
- removed DA3: NCP583XVxx, SOT,_TO:SOT563, symbol Regulators:NCP583XVxx
- removed DA4: NCP583SQxx, SOT,_TO:SC82AB, symbol Regulators:NCP583SQxx
- removed R5: 100k, Resistors:RES0603, symbol Resistors:R_0603
- removed fus2: Fuse, PCB_details:FuseSolder, symbol PCB_details:Fuse
- added R1: 100k, Resistors:RES0603, symbol Resistors:R_0603
- added XP5: 5Vin, Connectors:for_PolarOut_PLS2-2, symbol Connectors:for_PolarOut
- DA1: value MCP1700T-3302E -> MCP1700T
- SB2: renamed from SB1; value WKUP -> ON/WKUP
- XP2: Step h 2.54mm -> h 2mm
- XS1: renamed from XS4; Step h 2.54mm -> h 2mm
- renumbered C11 to C1, C7 to C10, C9 to C11, C10 to C12, C18 to C13, C19 to C14, C20 to C15, C13 to C16, C14 to C17, C15 to C18, C16 to C19, C12 to C2, C17 to C20, C8 to C3, C1 to C4, C2 to C5, C3 to C6, C4 to C7, C5 to C8, C6 to C9, DA6 to DA2, DA2 to DA3, DA5 to DA4, R8 to R10, R10 to R11, R11 to R12, R12 to R13, R13 to R14, R14 to R15, R1 to R2, R2 to R3, R6 to R4, R3 to R5, R4 to R6, R7 to R8, SB2 to SB1, VD6 to VD3, VD3 to VD4, VD4 to VD5, VD5 to VD6, XS1 to XS2, XS2 to XS3, XS3 to XS4
Connections:
- net +3.3V: now also R1.1
- net +USBvcc: now also XP5.1 (+/vcc)
- net ADC: now also DD1.14 (PB1/T3C4/T14C1/T1C3N/ADC9); no longer DD1.12 (ADC6/MISO1/T3C1/T16C1/PA6)
- net EN_WKUP: now also R1.2
- net GND: now also XP5.2 (-/gnd)
- net USER: now also DD1.12 (ADC6/MISO1/T3C1/T16C1/PA6); no longer DD1.14 (PB1/T3C4/T14C1/T1C3N/ADC9)
- net PWM renamed LoadCtrl
Other:
- moved on the sheet: C1, C10, C11, C12, C13, C14, C15, C16, C17, C18, C19, C2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

Commit message: Игровой таймер: компоненты расставлены
Parts:
- removed SB1: Down, Buttons,_Switches:BTN_5x5(AJ-037), symbol Switches:Button
- removed SB3: Up, Buttons,_Switches:BTN_5x5(AJ-037), symbol Switches:Button
- added C21: 0.1u, Capacitors:CAP0603, symbol Capacitors:C_0603
- added VD7: PESD3V3U1UB, Diodes:SOD523, symbol Protection:PESD3V3U1UB
- added fus2: Out | Vin, PCB_details:FuseSolder_x2_0603, symbol PCB_details:Fuse_x2
- renumbered SB2 to SB1
Connections:
- net +3.3V: now also fus2.3; no longer C4.1, XP1.1 (VCC)
- net +LOAD_OUT: now also fus2.2
- net LoadCtrl: now also DD1.12 (ADC6/MISO1/T3C1/T16C1/PA6); no longer DD1.13 (ADC7/MOSI1/T3C2/T14C1/T1C1N/T17C1/PA7)
- net USER: now also DD1.13 (ADC7/MOSI1/T3C2/T14C1/T1C1N/T17C1/PA7); no longer C12.1, DD1.12 (ADC6/MISO1/T3C1/T16C1/PA6), R12.1, R6.2
- net at R4.1, VU1.1 (A): now also VD7.C
- net at R4.2, XP2.1 (+/vcc): now also C21.1
- net at VU1.2 (C), XP2.2 (-/gnd): now also C21.2, VD7.A
- net BTN1: no longer names the net of DD1.10 (ADC4/NSS1/T14C1/PA4)
- net BTN2 renamed BATT_MEAS
- net BATT_MEAS: now also C12.1, R12.1, R6.2
- new net +USER_VCC: C4.1, XP1.1 (VCC), fus2.1
- no-connect marks 4 -> 5
Other:
- moved on the sheet: C11, C12, C3, HL1, R1, R10, R11, R12, R13, R3, R4, R5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

Commit message: GameTimer: работа завершена
Other:
- note added: "Start for Wkup btn\n(set to Bottom)"
- note removed: "Start for Wkuup btn\n(set to Bottom)"
Changed lines of the file:
@@
 EN_WKUP
 Text Notes 1450 6050 0    59   ~ 0
-Start for Wkuup btn\n(set to Bottom)
+Start for Wkup btn\n(set to Bottom)
 $Comp
 L Regulators:MCP1700T-xx02E DA1
